Commit message: Execution: gripper factory, OnRobot 2FG7, constraints/config handlers; new programs; launch and MoveIt config updates

File: src/ros2_SimRealRobotControl/ros2srrc_endeffectors/robotiq_hande/urdf/robotiq_hande_macro.urdf.xacro (robot description, xacro)
@@ -144,5 +144,5 @@
       <child link="robotiq_hande_left_finger"/>
       <axis xyz="-1 0 0"/>
-      <limit effort="130" lower="-0.0001" upper="0.0251" velocity="0.15"/>
+      <limit effort="130" lower="-0.0001" upper="0.05" velocity="0.15"/>
     </joint>
     <!-- Robotiq: right finger -->
@@ -174,5 +174,5 @@
       <child link="robotiq_hande_right_finger"/>
       <axis xyz="1 0 0"/>
-      <limit effort="130" lower="-0.0001" upper="0.0251" velocity="0.15"/>
+      <limit effort="130" lower="-0.0001" upper="0.05" velocity="0.15"/>
     </joint>
     <!-- SMALL CUBE FOR GRIPPER PLUGIN -->
@@ -189,8 +189,9 @@
       </visual>
     </link>
+    <!-- TCP frame aligned with robotiq_2f85 (ur5_2): same orientation relative to tool0 so same pose commands give same finger direction -->
     <joint name="EE_robotiq_hande_joint" type="fixed" >
       <parent link="robotiq_hande_base_link" />
       <child link="EE_robotiq_hande" />
-      <origin xyz="0.0 0.0 0.135" rpy="0 0 0"/>
+      <origin xyz="0.0 0.0 0.135" rpy="0 ${-pi/2} ${-pi/2}"/>
     </joint>
     <gazebo reference="EE_robotiq_hande_joint">

File: src/ros2_SimRealRobotControl/ros2srrc_endeffectors/robotiq_hande/urdf/robotiq_handev2_macro.urdf.xacro (robot description, xacro)
@@ -144,5 +144,5 @@
       <child link="robotiq_hande_left_finger"/>
       <axis xyz="-1 0 0"/>
-      <limit effort="130" lower="-0.0001" upper="0.0251" velocity="0.15"/>
+      <limit effort="130" lower="-0.0001" upper="0.05" velocity="0.15"/>
     </joint>
     <!-- Robotiq: right finger -->
@@ -174,5 +174,5 @@
       <child link="robotiq_hande_right_finger"/>
       <axis xyz="1 0 0"/>
-      <limit effort="130" lower="-0.0001" upper="0.0251" velocity="0.15"/>
+      <limit effort="130" lower="-0.0001" upper="0.05" velocity="0.15"/>
     </joint>
     <!-- SMALL CUBE FOR GRIPPER PLUGIN -->
