Commit message: Real robot: scaled controller, limits epsilon, 2FG7 port 50003, MoveIt/execution fixes

File: src/ros2_SimRealRobotControl/ros2srrc_endeffectors/robotiq_2f85/urdf/robotiq_2f85_macro.urdf.xacro (robot description, xacro)
@@ -3,4 +3,8 @@
   <!-- XACRO-MACRO of Robotiq 2f-85: -->
   <xacro:macro name="robotiq_2f85" params="bringup parent_link">
+    <!-- Material used by finger pad links (must be defined for URDF parser) -->
+    <material name="black">
+      <color rgba="0.1 0.1 0.1 1"/>
+    </material>
     <xacro:unless value="${bringup}">
       <!-- Robotiq 2f-85 TRANSMISSION: -->
@@ -78,7 +82,7 @@
         <mass value="0.018491" />
         <origin xyz="0.0 0.0 0.0" />
-        <inertia ixx = "0.000009" ixy = "-0.000001" ixz = "0.000000"
-            iyx = "-0.000001" iyy = "0.000001" iyz = "0.000000"
-            izx = "0.000000" izy = "0.000000" izz = "0.000010" />
+        <inertia ixx="0.000009" ixy="0.0" ixz="0.0"
+            iyy="0.000006" iyz="0.0"
+            izz="0.000010" />
       </inertial>
     </link>
@@ -106,7 +110,7 @@
         <mass value="0.018491" />
         <origin xyz="0.0 0.0 0.0" />
-        <inertia ixx = "0.000009" ixy = "-0.000001" ixz = "0.000000"
-            iyx = "-0.000001" iyy = "0.000001" iyz = "0.000000"
-            izx = "0.000000" izy = "0.000000" izz = "0.000010" />
+        <inertia ixx="0.000009" ixy="0.0" ixz="0.0"
+            iyy="0.000006" iyz="0.0"
+            izz="0.000010" />
       </inertial>
     </link>
@@ -395,4 +399,9 @@
         </geometry>
       </visual>
+      <collision>
+        <geometry>
+          <box size="0.001 0.001 0.001"/>
+        </geometry>
+      </collision>
     </link>
     <joint name="EE_robotiq_2f85_joint" type="fixed" >

File: src/ros2_SimRealRobotControl/ros2srrc_robots/ur5/urdf/ur5_common.xacro (robot description, xacro)
@@ -78,9 +78,11 @@
     <xacro:property name="shoulder_pan_velocity_limit" value="3.1416" scope="parent"/>
     <xacro:property name="shoulder_pan_effort_limit" value="150.0" scope="parent"/>
-    <xacro:property name="shoulder_lift_lower_limit" value="-1.5707" scope="parent"/>
+    <!-- Epsilon below -pi/2 so small negative noise is not out of bounds (Pilz/limits check) -->
+    <xacro:property name="shoulder_lift_lower_limit" value="-1.58" scope="parent"/>
     <xacro:property name="shoulder_lift_upper_limit" value="3.1416" scope="parent"/>
     <xacro:property name="shoulder_lift_velocity_limit" value="3.1416" scope="parent"/>
     <xacro:property name="shoulder_lift_effort_limit" value="150.0" scope="parent"/>
-    <xacro:property name="elbow_joint_lower_limit" value="0.0" scope="parent"/>
+    <!-- Epsilon below 0 so small negative noise (e.g. -2.396e-05) is not out of bounds (Pilz/limits check) -->
+    <xacro:property name="elbow_joint_lower_limit" value="-0.01" scope="parent"/>
     <xacro:property name="elbow_joint_upper_limit" value="3.1416" scope="parent"/>
     <xacro:property name="elbow_joint_velocity_limit" value="3.1416" scope="parent"/>

File: src/ros2_SimRealRobotControl/ros2srrc_robots/ur5/urdf/ur5_ros2control.xacro (robot description, xacro)
@@ -195,8 +195,8 @@
         </state_interface>
       </joint>
-      <!-- ELBOW JOINT -->
+      <!-- ELBOW JOINT (min -0.01 for consistency with URDF limit; avoids out-of-bounds on small negative noise) -->
       <joint name="elbow_joint">
         <command_interface name="position">
-          <param name="min">0.0</param>
+          <param name="min">-0.01</param>
           <param name="max">${pi}</param>
         </command_interface>
