Commit message: Fixed Table size

File: src/ros2_SimRealRobotControl/packages/ros2srrc_ur5/urdf/ur5.urdf.xacro (robot description, xacro)
@@ -68,5 +68,5 @@
   <!-- World: LINK -->
   <link name="world"/>
-  <!-- Robot Stand: LINK -->
+  <!-- Robot Stand: LINK (length X=184.4cm, width Y=84cm, height Z=50cm) -->
   <link name='robot_stand'>
     <inertial>
@@ -78,5 +78,5 @@
       <origin xyz="0 0 0" rpy=" 0 0 0"/>
       <geometry>
-        <box size = "0.2 0.2 0.5"/>
+        <box size = "1.844 0.84 0.5"/>
       </geometry>
     </collision>
@@ -84,5 +84,5 @@
       <origin xyz="0 0 0" rpy=" 0 0 0"/>
       <geometry>
-        <box size = "0.2 0.2 0.5"/>
+        <box size = "1.844 0.84 0.5"/>
       </geometry>
     </visual>
@@ -94,9 +94,9 @@
     <origin xyz="0.0 0.0 0.25" rpy="0.0 0.0 0.0" />
   </joint>
-  <!-- Robot Stand: Robot+Stand JOINT -->
+  <!-- Robot base: 31cm from bottom (-X) edge, 11.2cm from left (+Y) edge -->
   <joint name="stand_joint" type="fixed">
     <parent link= "robot_stand" />
     <child link = "base_link" />
-    <origin xyz="0.0 0.0 0.255" rpy="0.0 0.0 0.0" />
+    <origin xyz="-0.612 0.0 0.255" rpy="0.0 0.0 0.0" />
   </joint>
 </robot>

File: src/ros2_SimRealRobotControl/packages/ros2srrc_ur5/urdf/ur5_robotiq_2f85.urdf.xacro (robot description, xacro)
@@ -76,5 +76,5 @@
   <!-- World: LINK -->
   <link name="world"/>
-  <!-- Robot Stand: LINK -->
+  <!-- Robot Stand: LINK (length X=184.4cm, width Y=84cm, height Z=50cm) -->
   <link name='robot_stand'>
     <inertial>
@@ -86,5 +86,5 @@
       <origin xyz="0 0 0" rpy=" 0 0 0"/>
       <geometry>
-        <box size = "0.2 0.2 0.5"/>
+        <box size = "1.844 0.84 0.5"/>
       </geometry>
     </collision>
@@ -92,5 +92,5 @@
       <origin xyz="0 0 0" rpy=" 0 0 0"/>
       <geometry>
-        <box size = "0.2 0.2 0.5"/>
+        <box size = "1.844 0.84 0.5"/>
       </geometry>
     </visual>
@@ -102,9 +102,9 @@
     <origin xyz="0.0 0.0 0.25" rpy="0.0 0.0 0.0" />
   </joint>
-  <!-- Robot Stand: Robot+Stand JOINT -->
+  <!-- Robot base: 31cm from bottom (+X) edge, 11.2cm from left (+Y) edge -->
   <joint name="stand_joint" type="fixed">
     <parent link= "robot_stand" />
     <child link = "base_link" />
-    <origin xyz="0.0 0.0 0.255" rpy="0.0 0.0 0.0" />
+    <origin xyz="-0.612 0.0 0.255" rpy="0.0 0.0 0.0" />
   </joint>
 </robot>

File: src/ros2_SimRealRobotControl/packages/ros2srrc_ur5/urdf/ur5_robotiq_hande.urdf.xacro (robot description, xacro)
@@ -76,5 +76,5 @@
   <!-- World: LINK -->
   <link name="world"/>
-  <!-- Robot Stand: LINK -->
+  <!-- Robot Stand: LINK (length X=184.4cm, width Y=84cm, height Z=50cm) -->
   <link name='robot_stand'>
     <inertial>
@@ -86,5 +86,5 @@
       <origin xyz="0 0 0" rpy=" 0 0 0"/>
       <geometry>
-        <box size = "0.2 0.2 0.5"/>
+        <box size = "1.844 0.84 0.5"/>
       </geometry>
     </collision>
@@ -92,5 +92,5 @@
       <origin xyz="0 0 0" rpy=" 0 0 0"/>
       <geometry>
-        <box size = "0.2 0.2 0.5"/>
+        <box size = "1.844 0.84 0.5"/>
       </geometry>
     </visual>
@@ -102,9 +102,9 @@
     <origin xyz="0.0 0.0 0.25" rpy="0.0 0.0 0.0" />
   </joint>
-  <!-- Robot Stand: Robot+Stand JOINT -->
+  <!-- Robot base: 31cm from bottom (+X) edge, 11.2cm from left (+Y) edge -->
   <joint name="stand_joint" type="fixed">
     <parent link= "robot_stand" />
     <child link = "base_link" />
-    <origin xyz="0.0 0.0 0.255" rpy="0.0 0.0 0.0" />
+    <origin xyz="-0.612 0.0 0.255" rpy="0.0 0.0 0.0" />
   </joint>
 </robot>
