Commit message: Add OnRobot 2FG7 real-robot stack and speed up Hanoi pick/place.
Integrate onrobot driver/description packages, UR bringup, and gripper
backends so UR5+2FG7 can run pick-place and Tower of Hanoi on hardware.
Hanoi uses in-process pick/place, shorter pose publish, and MoveIt obstacle
clearing for reliable outer-peg picks without a center transit detour.

Co-authored-by: Cursor <cursoragent@cursor.com>

File: src/ros2_SimRealRobotControl/packages/ros2srrc_ur5/urdf/ur5.urdf.xacro (robot description, xacro)
@@ -68,5 +68,5 @@
   <!-- World: LINK -->
   <link name="world"/>
-  <!-- Robot Stand: LINK (length X=184.4cm, width Y=84cm, height Z=50cm) -->
+  <!-- Robot Stand: LINK (length X=84cm, width Y=184.4cm, height Z=84cm; top surface at z=0.84m) -->
   <link name='robot_stand'>
     <inertial>
@@ -78,5 +78,5 @@
       <origin xyz="0 0 0" rpy=" 0 0 0"/>
       <geometry>
-        <box size = "1.844 0.84 0.5"/>
+        <box size = "0.84 1.844 0.84"/>
       </geometry>
     </collision>
@@ -84,5 +84,5 @@
       <origin xyz="0 0 0" rpy=" 0 0 0"/>
       <geometry>
-        <box size = "1.844 0.84 0.5"/>
+        <box size = "0.84 1.844 0.84"/>
       </geometry>
     </visual>
@@ -92,11 +92,11 @@
     <parent link= "world" />
     <child link = "robot_stand" />
-    <origin xyz="0.0 0.0 0.25" rpy="0.0 0.0 0.0" />
+    <origin xyz="0.0 0.0 0.42" rpy="0.0 0.0 0.0" />
   </joint>
-  <!-- Robot base: 31cm from bottom (-X) edge, 11.2cm from left (+Y) edge -->
+  <!-- Robot base: 31cm from bottom (-Y) edge, centered on short (X) axis -->
   <joint name="stand_joint" type="fixed">
     <parent link= "robot_stand" />
     <child link = "base_link" />
-    <origin xyz="-0.612 0.0 0.255" rpy="0.0 0.0 0.0" />
+    <origin xyz="0.0 -0.612 0.425" rpy="0.0 0.0 0.0" />
   </joint>
 </robot>

File: src/ros2_SimRealRobotControl/packages/ros2srrc_ur5/urdf/ur5_robotiq_2f85.urdf.xacro (robot description, xacro)
@@ -76,5 +76,5 @@
   <!-- World: LINK -->
   <link name="world"/>
-  <!-- Robot Stand: LINK (length X=184.4cm, width Y=84cm, height Z=50cm) -->
+  <!-- Robot Stand: LINK (length X=84cm, width Y=184.4cm, height Z=84cm; top surface at z=0.84m) -->
   <link name='robot_stand'>
     <inertial>
@@ -86,5 +86,5 @@
       <origin xyz="0 0 0" rpy=" 0 0 0"/>
       <geometry>
-        <box size = "1.844 0.84 0.5"/>
+        <box size = "0.84 1.844 0.84"/>
       </geometry>
     </collision>
@@ -92,5 +92,5 @@
       <origin xyz="0 0 0" rpy=" 0 0 0"/>
       <geometry>
-        <box size = "1.844 0.84 0.5"/>
+        <box size = "0.84 1.844 0.84"/>
       </geometry>
     </visual>
@@ -100,11 +100,11 @@
     <parent link= "world" />
     <child link = "robot_stand" />
-    <origin xyz="0.0 0.0 0.25" rpy="0.0 0.0 0.0" />
+    <origin xyz="0.0 0.0 0.42" rpy="0.0 0.0 0.0" />
   </joint>
-  <!-- Robot base: 31cm from bottom (+X) edge, 11.2cm from left (+Y) edge -->
+  <!-- Robot base: 31cm from bottom (-Y) edge, centered on short (X) axis -->
   <joint name="stand_joint" type="fixed">
     <parent link= "robot_stand" />
     <child link = "base_link" />
-    <origin xyz="-0.612 0.0 0.255" rpy="0.0 0.0 0.0" />
+    <origin xyz="0.0 -0.612 0.425" rpy="0.0 0.0 0.0" />
   </joint>
 </robot>

File: src/ros2_SimRealRobotControl/packages/ros2srrc_ur5/urdf/ur5_robotiq_hande.urdf.xacro (robot description, xacro)
@@ -76,5 +76,5 @@
   <!-- World: LINK -->
   <link name="world"/>
-  <!-- Robot Stand: LINK (length X=184.4cm, width Y=84cm, height Z=50cm) -->
+  <!-- Robot Stand: LINK (length X=84cm, width Y=184.4cm, height Z=84cm; top surface at z=0.84m) -->
   <link name='robot_stand'>
     <inertial>
@@ -86,5 +86,5 @@
       <origin xyz="0 0 0" rpy=" 0 0 0"/>
       <geometry>
-        <box size = "1.844 0.84 0.5"/>
+        <box size = "0.84 1.844 0.84"/>
       </geometry>
     </collision>
@@ -92,5 +92,5 @@
       <origin xyz="0 0 0" rpy=" 0 0 0"/>
       <geometry>
-        <box size = "1.844 0.84 0.5"/>
+        <box size = "0.84 1.844 0.84"/>
       </geometry>
     </visual>
@@ -100,11 +100,11 @@
     <parent link= "world" />
     <child link = "robot_stand" />
-    <origin xyz="0.0 0.0 0.25" rpy="0.0 0.0 0.0" />
+    <origin xyz="0.0 0.0 0.42" rpy="0.0 0.0 0.0" />
   </joint>
-  <!-- Robot base: 31cm from bottom (+X) edge, 11.2cm from left (+Y) edge -->
+  <!-- Robot base: 31cm from bottom (-Y) edge, centered on short (X) axis -->
   <joint name="stand_joint" type="fixed">
     <parent link= "robot_stand" />
     <child link = "base_link" />
-    <origin xyz="-0.612 0.0 0.255" rpy="0.0 0.0 0.0" />
+    <origin xyz="0.0 -0.612 0.425" rpy="0.0 0.0 0.0" />
   </joint>
 </robot>

File: src/ros2_SimRealRobotControl/ros2srrc_robots/ur5/urdf/ur5_ros2control.xacro (robot description, xacro)
@@ -155,5 +155,5 @@
         </sensor>
       </xacro:if>
-      <!-- SHOULDER PAN JOINT -->
+      <!-- SHOULDER PAN JOINT (initial: 90° ready pose over +Y table) -->
       <joint name="shoulder_pan_joint">
         <command_interface name="position">
@@ -166,5 +166,5 @@
         </command_interface>
         <state_interface name="position">
-          <param name="initial_value">0.0</param>
+          <param name="initial_value">${pi/2}</param>
         </state_interface>
         <state_interface name="velocity">
@@ -206,5 +206,5 @@
         </command_interface>
         <state_interface name="position">
-          <param name="initial_value">0.0</param>
+          <param name="initial_value">${pi/2}</param>
         </state_interface>
         <state_interface name="velocity">
@@ -246,5 +246,5 @@
         </command_interface>
         <state_interface name="position">
-          <param name="initial_value">0.0</param>
+          <param name="initial_value">${-pi/2}</param>
         </state_interface>
         <state_interface name="velocity">
